File: Firefly-Box.sch (EAGLE design)
At the start: 35 parts, among them J1 USB MICRO, U1 ATMEGA32U4-XUMU, U2 ATMEGA32U4-XUAU, Y1 16MHz KX-7

Commit message: Add Box headers
Parts:
- removed J1: USB MICRO, SmartPrj:MYCON2_USB-MINI-B
- added CONN2: CONN_USB, dp_devices:CONN_USB
- added JP1, JP2: (no value), pinhead:PINHD-1X15
- added JP3: (no value), pinhead:PINHD-1X14
- added JP4, JP5: (no value), pinhead:PINHD-1X4
Connections:
- removed net USBID: J1.ID
- removed net XUSB: J1.VBUS
- new net 5V: CONN2USB.VUSB, U1.VBUS
- net D+: now also CONN2USB.D+; no longer J1.D+
- net D-: now also CONN2USB.D-; no longer J1.D-
- net GND: now also CONN2USB.GND; no longer J1.GND, J1.SH1, J1.SH2, J1.SH3, J1.SH4, J1.SH5, J1.SH6
- net VUSB: no longer U1.VBUS
Changed lines of the file:
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@@
 <layer number="97" name="Info" color="7" fill="1" visible="yes" active="yes"/>
 <layer number="98" name="Guide" color="6" fill="1" visible="yes" active="yes"/>
+<layer number="99" name="SpiceOrder" color="5" fill="1" visible="yes" active="yes"/>
 <layer number="100" name="Muster" color="7" fill="1" visible="yes" active="yes"/>
 <layer number="101" name="Patch_Top" color="7" fill="1" visible="yes" active="yes"/>
@@
 <part name="GND17" library="supply1" deviceset="GND" device=""/>
 <part name="R1" library="SmartPrj" deviceset="R-EU_" device="R0603" value="1M"/>
-<part name="U$25" library="MyPOW" deviceset="VUSB" device=""/>
 <part name="SUPPLY2" library="supply2" deviceset="GND1" device="" value="UGND"/>
 <part name="U$30" library="MyPOW" deviceset="COM" device=""/>
@@
 <part name="Y1" library="SmartPrj" deviceset="CRYSTAL-3.2-2.5" device="" value="16MHz KX-7"/>
 <part name="D2" library="diode" deviceset="DIODE-" device="MINIMELF" value="CD1206-S01575"/>
-<part name="J1" library="SmartPrj" deviceset="MYCON2_USB-MINI-B" device="" value="USB MICRO"/>
 <part name="GND2" library="supply1" deviceset="GND" device=""/>
 <part name="R4" library="GadgetFactory_6.0" deviceset="R" device="0805" value="22R"/>
@@
 <part name="R10" library="GadgetFactory_6.0" deviceset="R" device="0805" value="1K"/>
 <part name="R11" library="GadgetFactory_6.0" deviceset="R" device="0805" value="1K"/>
+<part name="CONN2" library="dp_devices" deviceset="CONN_USB" device=""/>
+<part name="JP1" library="pinhead" deviceset="PINHD-1X15" device=""/>
+<part name="JP2" library="pinhead" deviceset="PINHD-1X15" device=""/>
+<part name="JP3" library="pinhead" deviceset="PINHD-1X14" device=""/>
+<part name="JP4" library="pinhead" deviceset="PINHD-1X4" device=""/>
+<part name="JP5" library="pinhead" deviceset="PINHD-1X4" device=""/>
 </parts>
 <sheets>
@@
 <attribute name="NAME" x="66.294" y="78.74" size="1.778" layer="95" rot="R180"/>
 </instance>
+<instance part="JP1" gate="A" x="55.88" y="121.92" rot="R90"/>
+<instance part="JP2" gate="A" x="236.22" y="96.52" rot="R180"/>
+<instance part="JP3" gate="A" x="203.2" y="81.28" rot="R90"/>
+<instance part="JP4" gate="A" x="22.86" y="104.14"/>
+<instance part="JP5" gate="A" x="22.86" y="83.82"/>
 </instances>
 <busses>
@@
 <attribute name="VALUE" x="-73.025" y="111.252" size="1.778" layer="96" rot="R180"/>
 </instance>
-<instance part="U$25" gate="G$1" x="-38.1" y="66.04"/>
 <instance part="SUPPLY2" gate="G$1" x="-63.5" y="38.1"/>
 <instance part="U$30" gate="G$1" x="-30.48" y="66.04"/>
@@
 <attribute name="VALUE" x="-68.8086" y="119.38" size="1.778" layer="96" rot="R90"/>
 </instance>
-<instance part="J1" gate="G$1" x="-114.3" y="-5.08" rot="MR0"/>
-<instance part="GND2" gate="1" x="-88.9" y="-58.42"/>
+<instance part="GND2" gate="1" x="-129.54" y="-55.88"/>
 <instance part="R4" gate="A" x="-60.96" y="0"/>
 <instance part="R5" gate="A" x="-60.96" y="-7.62"/>
@@
 <instance part="R10" gate="A" x="292.1" y="-35.56" rot="R270"/>
 <instance part="R11" gate="A" x="335.28" y="-38.1" rot="R270"/>
+<instance part="CONN2" gate="USB" x="-116.84" y="-2.54"/>
 </instances>
 <busses>
@@
 </segment>
 <segment>
-<wire x1="-127" y1="-10.16" x2="-132.08" y2="-10.16" width="0.1524" layer="91"/>
-<wire x1="-132.08" y1="-7.62" x2="-132.08" y2="-10.16" width="0.1524" layer="91"/>
-<wire x1="-127" y1="-7.62" x2="-132.08" y2="-7.62" width="0.1524" layer="91"/>
-<wire x1="-132.08" y1="-5.08" x2="-132.08" y2="-7.62" width="0.1524" layer="91"/>
-<wire x1="-127" y1="-5.08" x2="-132.08" y2="-5.08" width="0.1524" layer="91"/>
-<wire x1="-132.08" y1="-2.54" x2="-132.08" y2="-5.08" width="0.1524" layer="91"/>
-<wire x1="-127" y1="-2.54" x2="-132.08" y2="-2.54" width="0.1524" layer="91"/>
-<wire x1="-121.92" y1="-22.86" x2="-132.08" y2="-22.86" width="0.1524" layer="91"/>
-<wire x1="-132.08" y1="-22.86" x2="-132.08" y2="-15.24" width="0.1524" layer="91"/>
-<wire x1="-132.08" y1="-15.24" x2="-132.08" y2="-12.7" width="0.1524" layer="91"/>
-<wire x1="-132.08" y1="-12.7" x2="-132.08" y2="-10.16" width="0.1524" layer="91"/>
-<wire x1="-88.9" y1="-55.88" x2="-132.08" y2="-55.88" width="0.1524" layer="91"/>
-<wire x1="-132.08" y1="-55.88" x2="-132.08" y2="-22.86" width="0.1524" layer="91"/>
-<wire x1="-127" y1="-12.7" x2="-132.08" y2="-12.7" width="0.1524" layer="91"/>
-<wire x1="-127" y1="-15.24" x2="-132.08" y2="-15.24" width="0.1524" layer="91"/>
-<junction x="-132.08" y="-7.62"/>
-<junction x="-132.08" y="-5.08"/>
-<junction x="-132.08" y="-10.16"/>
-<junction x="-132.08" y="-22.86"/>
-<junction x="-132.08" y="-12.7"/>
-<junction x="-132.08" y="-15.24"/>
-<label x="-129.54" y="-2.54" size="1.778" layer="95" rot="MR0"/>
-<label x="-129.54" y="-22.86" size="1.778" layer="95"/>
-<pinref part="J1" gate="G$1" pin="SH1"/>
-<pinref part="J1" gate="G$1" pin="SH2"/>
-<pinref part="J1" gate="G$1" pin="SH3"/>
-<pinref part="J1" gate="G$1" pin="SH4"/>
-<pinref part="J1" gate="G$1" pin="SH5"/>
-<pinref part="J1" gate="G$1" pin="SH6"/>
 <pinref part="GND2" gate="1" pin="GND"/>
-<pinref part="J1" gate="G$1" pin="GND"/>
-<wire x1="-101.6" y1="-10.16" x2="-88.9" y2="-10.16" width="0.1524" layer="91"/>
-<wire x1="-88.9" y1="-10.16" x2="-88.9" y2="-55.88" width="0.1524" layer="91"/>
+<wire x1="-129.54" y1="-20.32" x2="-129.54" y2="-53.34" width="0.1524" layer="91"/>
+<wire x1="-129.54" y1="-20.32" x2="-129.54" y2="10.16" width="0.2032" layer="91"/>
+<pinref part="CONN2" gate="USB" pin="GND"/>
+<wire x1="-129.54" y1="10.16" x2="-111.76" y2="10.16" width="0.2032" layer="91"/>
+<wire x1="-111.76" y1="10.16" x2="-111.76" y2="2.54" width="0.2032" layer="91"/>
 </segment>
 </net>
@@
 <wire x1="-68.58" y1="-2.54" x2="-66.04" y2="0" width="0.1524" layer="91"/>
 <label x="-86.36" y="-2.54" size="1.778" layer="95" rot="MR0"/>
-<pinref part="J1" gate="G$1" pin="D-"/>
 <pinref part="R4" gate="A" pin="1"/>
+<pinref part="CONN2" gate="USB" pin="D-"/>
+<wire x1="-101.6" y1="-2.54" x2="-111.76" y2="-2.54" width="0.2032" layer="91"/>
 </segment>
 </net>
@@
 <wire x1="-66.04" y1="-5.08" x2="-66.04" y2="-7.62" width="0.1524" layer="91"/>
 <label x="-86.36" y="-5.08" size="1.778" layer="95" rot="MR0"/>
-<pinref part="J1" gate="G$1" pin="D+"/>
 <pinref part="R5" gate="A" pin="1"/>
+<pinref part="CONN2" gate="USB" pin="D+"/>
+<wire x1="-101.6" y1="-5.08" x2="-111.76" y2="-5.08" width="0.2032" layer="91"/>
 </segment>
 </net>
@@
 </segment>
 </net>
-<net name="XUSB" class="3">
+<net name="5V" class="3">
 <segment>
 <wire x1="-81.28" y1="0" x2="-81.28" y2="10.16" width="0.1524" layer="91"/>
@@
 <label x="-91.44" y="0" size="1.778" layer="95" rot="MR0"/>
 <label x="-78.74" y="10.16" size="1.778" layer="95"/>
-<pinref part="J1" gate="G$1" pin="VBUS"/>
+<pinref part="CONN2" gate="USB" pin="VUSB"/>
+<wire x1="-101.6" y1="0" x2="-111.76" y2="0" width="0.2032" layer="91"/>
+</segment>
+<segment>
+<wire x1="-7.62" y1="71.12" x2="-27.94" y2="71.12" width="0.1524" layer="91"/>
+<wire x1="-27.94" y1="71.12" x2="-27.94" y2="58.42" width="0.1524" layer="91"/>
+<wire x1="-27.94" y1="58.42" x2="-38.1" y2="58.42" width="0.1524" layer="91"/>
+<wire x1="-38.1" y1="58.42" x2="-38.1" y2="63.5" width="0.1524" layer="91"/>
+<label x="-35.56" y="58.42" size="1.778" layer="95"/>
+<pinref part="U1" gate="G$1" pin="VBUS"/>
 </segment>
 </net>
@@
 <net name="VUSB" class="0">
 <segment>
-<wire x1="-7.62" y1="71.12" x2="-27.94" y2="71.12" width="0.1524" layer="91"/>
-<wire x1="-27.94" y1="71.12" x2="-27.94" y2="58.42" width="0.1524" layer="91"/>
-<wire x1="-27.94" y1="58.42" x2="-38.1" y2="58.42" width="0.1524" layer="91"/>
-<wire x1="-38.1" y1="58.42" x2="-38.1" y2="63.5" width="0.1524" layer="91"/>
-<label x="-35.56" y="58.42" size="1.778" layer="95"/>
-<pinref part="U$25" gate="G$1" pin="VUSB"/>
-<pinref part="U1" gate="G$1" pin="VBUS"/>
-</segment>
-<segment>
 <wire x1="149.86" y1="71.12" x2="129.54" y2="71.12" width="0.1524" layer="91"/>
 <label x="142.24" y="71.12" size="1.778" layer="95"/>
@@
 </segment>
 </net>
-<net name="USBID" class="0">
-<segment>
-<wire x1="-93.98" y1="-7.62" x2="-101.6" y2="-7.62" width="0.1524" layer="91"/>
-<label x="-93.98" y="-7.62" size="1.778" layer="95" rot="MR0"/>
-<pinref part="J1" gate="G$1" pin="ID"/>
-</segment>
-</net>
